File: pureModular/pureVCO/pureVCO.brd (EAGLE design)
At the start: 68.8 x 100 mm, 118 parts, among them IC1 TL072, IC2 TL072, IC3 TL072, IC4 TL072, IC5 TL072, IC6 TL072, IC7 TL072, IC8 LM4040A50IDBZT, T1 MMBFJ309

Commit message: VCO Updated to V3
Parts:
- added R54: 10k, GMSN:R0805
- COARSE: device GMSN:POTENTIOMETER_9MM -> GMSN:POT_9MM_RED_KNOB
- FINE: device GMSN:POTENTIOMETER_9MM -> GMSN:POT_9MM_RED_MXR_KNOB
- FM_LEVEL, PWM_LEVEL: device GMSN:POTENTIOMETER_9MM -> GMSN:POT_9MM_GREEN_KNOB
- PULSE_MIX, SAW_MIX, SINE_MIX, TRI_MIX: value B100k -> B10k; device GMSN:POTENTIOMETER_9MM -> GMSN:POT_9MM_BLUE_KNOB
- PULSE_WIDTH: device GMSN:POTENTIOMETER_9MM -> GMSN:POT_9MM_YELLOW_KNOB
- R45: value 10k -> 100k
- R46: value 19k1 -> 50k
- R47: value 1k3 -> 0R
- R48, R49, R50, R51, R52, R53: value 100k -> 10k
- TC1: device GMSN:0204/7 -> GMSN:0207/8.5
- moved R53 18.0 mm to (29.2, 38.1), turned to 90 degrees
- moved R52 1.27 mm to (11.4, 39.4)
Connections:
- removed net N$35: IC7.3, R48.2, R49.2, R50.2, R51.2
- new net N$26: IC7.6, R53.1, R54.2
- net GND: now also IC7.3, TP1.2; no longer R53.1, TP1.B1
- net N$10: now also TP1.1; no longer TP1.B2
- net N$12: now also TP1.6; no longer TP1.C2
- net N$13: now also TP1.3; no longer TP1.C1
- net N$14: now also TP2.6; no longer TP2.C2
- net N$18: now also TP1.4, TP1.5; no longer TP1.E1, TP1.E2
- net N$25: now also MIX.TIP, R53.2; no longer IC7.6
- net N$48: now also R48.2, R49.2, R50.2, R51.2; no longer R53.2
- net N$49: now also R54.1; no longer MIX.TIP
- net N$76: now also TP2.1; no longer TP2.B2
- net N$77: now also TP2.5; no longer TP2.E2
- net N$78: now also TP2.4; no longer TP2.E1
- net N$80: now also TP2.2; no longer TP2.B1
- net N$82: now also TP2.3; no longer TP2.C1
Routing:
- net N$48: track 7.07 -> 77.5 mm, vias 0 -> 4
- net N$35: track 69.4 -> 0.00 mm, vias 4 -> 0
- net N$25: track 1.27 -> 52.3 mm
- net N$49: track 33.9 -> 5.94 mm
- net N$26: track 0.00 -> 15.3 mm
- net N$4: track 66.0 -> 62.5 mm
- net N$1: track 13.2 -> 12.1 mm
- net N$37: track 10.2 -> 9.30 mm
- net N$16: track 19.1 -> 18.4 mm
- net N$7: track 31.1 -> 30.4 mm
- net N$10: track 36.9 -> 36.3 mm
- net N$20: track 28.5 -> 28.0 mm
Other:
- outline, holes or cut-outs redrawn
