File: pureModular/pureVCO/pureVCO.sch (EAGLE design)
At the start: 116 parts, among them IC1 TL072, IC2 TL072, IC3 TL072, IC4 TL072, IC5 TL072, IC6 TL072, IC7 TL072, IC8 LM4040A50IDBZT, T1 MMBFJ309

Commit message: VCO Updated to V3
Parts:
- added R54: 10k, GMSN:RESISTOR_USR0805
- COARSE: device GMSN:RESISTOR_VARIABLE9MM_POT -> GMSN:RESISTOR_VARIABLEPOT_9MM_RED_KNOB
- FINE: device GMSN:RESISTOR_VARIABLE9MM_POT -> GMSN:RESISTOR_VARIABLEPOT_9MM_RED_MXR_KNOB
- FM_LEVEL, PWM_LEVEL: device GMSN:RESISTOR_VARIABLE9MM_POT -> GMSN:RESISTOR_VARIABLEPOT_9MM_GREEN_KNOB
- PULSE_MIX, SAW_MIX, SINE_MIX, TRI_MIX: value B100k -> B10k; device GMSN:RESISTOR_VARIABLE9MM_POT -> GMSN:RESISTOR_VARIABLEPOT_9MM_BLUE_KNOB
- PULSE_WIDTH: device GMSN:RESISTOR_VARIABLE9MM_POT -> GMSN:RESISTOR_VARIABLEPOT_9MM_YELLOW_KNOB
- R45: value 10k -> 100k
- R46: value 19k1 -> 50k
- R47: value 1k3 -> 0R
- R48, R49, R50, R51, R52, R53: value 100k -> 10k
- TC1: device GMSN:RESISTOR_US0204/7 -> GMSN:RESISTOR_US0207/8.5
Connections:
- removed net N$35: IC7A.+IN, R48.2, R49.2, R50.2, R51.2
- new net N$26: IC7B.-IN, R53.1, R54.2
- net GND: now also IC7A.+IN; no longer R53.1
- net N$25: now also MIX.TIP, R53.2; no longer IC7B.-IN
- net N$48: now also R48.2, R49.2, R50.2, R51.2; no longer R53.2
- net N$49: now also R54.1; no longer MIX.TIP
Other:
- moved on the sheet: C4, C8, IC2B, IC7B, IC8, MIX, R12, R52, R53, R7, R8, SYNC
