File: pureModular/pureVCO/Pure VCO.brd (EAGLE design)
At the start: 68.8 x 100 mm, 119 parts, among them IC1 TL072, IC2 TL072, IC3 TL072, IC4 TL072, IC5 TL072, IC6 TL072, IC7 TL072, IC8 LM4040A50IDBZT, T1 MMBFJ309

Commit message: Minor corrections. Awaiting Testing. No ready for public consumption.
Parts:
- removed R54: 10k, GMSN:R0805
- COARSE: device GMSN:POT_9MM_RED_KNOB -> GMSN:POTENTIOMETER_9MM
- FINE: device GMSN:POT_9MM_RED_MXR_KNOB -> GMSN:POTENTIOMETER_9MM
- FM_LEVEL, PWM_LEVEL: device GMSN:POT_9MM_GREEN_KNOB -> GMSN:POTENTIOMETER_9MM
- PULSE_MIX, SAW_MIX, SINE_MIX, TRI_MIX: value B10k -> B100k; device GMSN:POT_9MM_BLUE_KNOB -> GMSN:POTENTIOMETER_9MM
- PULSE_WIDTH: device GMSN:POT_9MM_YELLOW_KNOB -> GMSN:POTENTIOMETER_9MM
- R48, R49, R50, R51, R52, R53: value 10k -> 100k
- TC1: device GMSN:0207/8.5 -> GMSN:0204/7
- moved R53 18.0 mm to (11.4, 35.6), turned to 0 degrees
- moved R52 1.27 mm to (12.7, 39.4)
Connections:
- removed net N$26: IC7.6, R53.1, R54.2
- new net N$35: IC7.3, R48.2, R49.2, R50.2, R51.2
- net GND: now also R53.1, TP1.B1; no longer IC7.3, TP1.2
- net N$10: now also TP1.B2; no longer TP1.1
- net N$12: now also TP1.C2; no longer TP1.6
- net N$13: now also TP1.C1; no longer TP1.3
- net N$14: now also TP2.C2; no longer TP2.6
- net N$18: now also TP1.E1, TP1.E2; no longer TP1.4, TP1.5
- net N$25: now also IC7.6; no longer MIX.TIP, R53.2
- net N$48: now also R53.2; no longer R48.2, R49.2, R50.2, R51.2
- net N$49: now also MIX.TIP; no longer R54.1
- net N$76: now also TP2.B2; no longer TP2.1
- net N$77: now also TP2.E2; no longer TP2.5
- net N$78: now also TP2.E1; no longer TP2.4
- net N$80: now also TP2.B1; no longer TP2.2
- net N$82: now also TP2.C1; no longer TP2.3
Routing:
- net N$48: track 77.5 -> 7.07 mm, vias 4 -> 0
- net N$35: track 0.00 -> 69.4 mm, vias 0 -> 4
- net N$25: track 52.3 -> 1.27 mm
- net N$49: track 5.94 -> 33.9 mm
- net N$26: track 15.3 -> 0.00 mm
- net N$4: track 62.5 -> 66.0 mm
- net N$1: track 12.1 -> 13.2 mm
- net N$37: track 9.30 -> 10.2 mm
- net N$16: track 18.4 -> 19.1 mm
- net N$7: track 30.4 -> 31.1 mm
- net N$10: track 36.3 -> 36.9 mm
- net N$20: track 28.0 -> 28.5 mm
Other:
- outline, holes or cut-outs redrawn

Commit message: VCO 3.1
Changed mixer from Average to Sum. Mixer outputs are now inversions of the individual out. Might be useful?
Resistor values around mixer reduced to 10k, inline with low noise techniques.
Parts:
- removed R53: 100k, GMSN:R0805
- COARSE: device GMSN:POTENTIOMETER_9MM -> GMSN:POT_9MM_RED_KNOB
- FINE: device GMSN:POTENTIOMETER_9MM -> GMSN:POT_9MM_RED_MXR_KNOB
- FM_LEVEL, PWM_LEVEL: device GMSN:POTENTIOMETER_9MM -> GMSN:POT_9MM_GREEN_KNOB
- PULSE_MIX, SAW_MIX, SINE_MIX, TRI_MIX: device GMSN:POTENTIOMETER_9MM -> GMSN:POT_9MM_BLUE_KNOB
- PULSE_WIDTH: device GMSN:POTENTIOMETER_9MM -> GMSN:POT_9MM_YELLOW_KNOB
- R48, R49, R50, R51, R52: value 100k -> 10k
- TC1: device GMSN:0204/7 -> GMSN:0207/8.5
Connections:
- removed net N$35: IC7.3, R48.2, R49.2, R50.2, R51.2
- net GND: now also IC7.3, TP1.2; no longer R53.1, TP1.B1
- net N$10: now also TP1.1; no longer TP1.B2
- net N$12: now also TP1.6; no longer TP1.C2
- net N$13: now also TP1.3; no longer TP1.C1
- net N$14: now also TP2.6; no longer TP2.C2
- net N$18: now also TP1.4, TP1.5; no longer TP1.E1, TP1.E2
- net N$48: now also R48.2, R49.2, R50.2, R51.2; no longer R53.2
- net N$76: now also TP2.1; no longer TP2.B2
- net N$77: now also TP2.5; no longer TP2.E2
- net N$78: now also TP2.4; no longer TP2.E1
- net N$80: now also TP2.2; no longer TP2.B1
- net N$82: now also TP2.3; no longer TP2.C1
Routing:
- net N$35: track 69.4 -> 0.00 mm, vias 4 -> 0
- net N$48: track 7.07 -> 75.1 mm, vias 0 -> 4
- net N$4: track 66.0 -> 62.5 mm
- net N$7: track 31.1 -> 29.7 mm
- net N$16: track 19.1 -> 18.4 mm
- net N$10: track 36.9 -> 36.4 mm
- net N$20: track 28.5 -> 28.0 mm
Other:
- board text added: "Pure VCO V3.1 cc-by 4.0 2021 The Little Red Hen"
- board text removed: "Pure VCO V3 cc-by 4.0 2018"
