File: pureModular/pureVCO/Pure VCO.sch (EAGLE design)
At the start: 117 parts, among them IC1 TL072, IC2 TL072, IC3 TL072, IC4 TL072, IC5 TL072, IC6 TL072, IC7 TL072, IC8 LM4040A50IDBZT, T1 MMBFJ309

Commit message: Minor corrections. Awaiting Testing. No ready for public consumption.
Parts:
- removed R54: 10k, GMSN:RESISTOR_USR0805
- COARSE: device GMSN:RESISTOR_VARIABLEPOT_9MM_RED_KNOB -> GMSN:RESISTOR_VARIABLE9MM_POT
- FINE: device GMSN:RESISTOR_VARIABLEPOT_9MM_RED_MXR_KNOB -> GMSN:RESISTOR_VARIABLE9MM_POT
- FM_LEVEL, PWM_LEVEL: device GMSN:RESISTOR_VARIABLEPOT_9MM_GREEN_KNOB -> GMSN:RESISTOR_VARIABLE9MM_POT
- PULSE_MIX, SAW_MIX, SINE_MIX, TRI_MIX: value B10k -> B100k; device GMSN:RESISTOR_VARIABLEPOT_9MM_BLUE_KNOB -> GMSN:RESISTOR_VARIABLE9MM_POT
- PULSE_WIDTH: device GMSN:RESISTOR_VARIABLEPOT_9MM_YELLOW_KNOB -> GMSN:RESISTOR_VARIABLE9MM_POT
- R48, R49, R50, R51, R52, R53: value 10k -> 100k
- TC1: device GMSN:RESISTOR_US0207/8.5 -> GMSN:RESISTOR_US0204/7
Connections:
- removed net N$26: IC7B.-IN, R53.1, R54.2
- new net N$35: IC7A.+IN, R48.2, R49.2, R50.2, R51.2
- net GND: now also R53.1; no longer IC7A.+IN
- net N$25: now also IC7B.-IN; no longer MIX.TIP, R53.2
- net N$48: now also R53.2; no longer R48.2, R49.2, R50.2, R51.2
- net N$49: now also MIX.TIP; no longer R54.1
Other:
- moved on the sheet: IC7B, MIX, R52, R53

Commit message: VCO 3.1
Changed mixer from Average to Sum. Mixer outputs are now inversions of the individual out. Might be useful?
Resistor values around mixer reduced to 10k, inline with low noise techniques.
Parts:
- removed R53: 100k, GMSN:RESISTOR_USR0805
- COARSE: device GMSN:RESISTOR_VARIABLE9MM_POT -> GMSN:RESISTOR_VARIABLEPOT_9MM_RED_KNOB
- FINE: device GMSN:RESISTOR_VARIABLE9MM_POT -> GMSN:RESISTOR_VARIABLEPOT_9MM_RED_MXR_KNOB
- FM_LEVEL, PWM_LEVEL: device GMSN:RESISTOR_VARIABLE9MM_POT -> GMSN:RESISTOR_VARIABLEPOT_9MM_GREEN_KNOB
- PULSE_MIX, SAW_MIX, SINE_MIX, TRI_MIX: device GMSN:RESISTOR_VARIABLE9MM_POT -> GMSN:RESISTOR_VARIABLEPOT_9MM_BLUE_KNOB
- PULSE_WIDTH: device GMSN:RESISTOR_VARIABLE9MM_POT -> GMSN:RESISTOR_VARIABLEPOT_9MM_YELLOW_KNOB
- R48, R49, R50, R51, R52: value 100k -> 10k
- TC1: device GMSN:RESISTOR_US0204/7 -> GMSN:RESISTOR_US0207/8.5
Connections:
- removed net N$35: IC7A.+IN, R48.2, R49.2, R50.2, R51.2
- net GND: now also IC7A.+IN; no longer R53.1
- net N$48: now also R48.2, R49.2, R50.2, R51.2; no longer R53.2
